File: Kicad/2ndDayPCB/2ndDayPCB.kicad_pcb (KiCad board)
At the start: 2 copper layers, 63.3 x 68.2 mm, 27 parts, among them SW1 SW_Push, SW2 SW_Push, SW3 SW_Push, U1 XIAO-ESP32-C3-DIP

Commit message: pcb changes
Other:
- board text added: "16"
- board text added: "Aryan India Gavaskar"
- board text added: "INDIA"
